Commit message: Send static transform now

File: lasertracker_ros2_control/description/urdf/lasertracker.urdf.xacro (robot description, xacro)
@@ -4,10 +4,5 @@
   <xacro:include filename="$(find lasertracker_ros2_control)/description/ros2_control/lasertracker.ros2_control.xacro" />
   <!-- Used for fixing sensor -->
-  <link name="world"/>
-  <link name="base_link"/>
-  <joint name="base_joint" type="fixed">
-    <parent link="world"/>
-    <child link="base_link" />
-  </joint>
+  <link name="lasertracker"/>
   <xacro:lasertracker_ros2_control/>
 </robot>
